Commit message: got adam hopping and hopper config and urdf modifications done.

File: resources/robots/adam/urdf/adam.urdf (robot description, URDF)
Before this commit: robot adam, 21 links, 20 joints
Links:
- removed link base_link
- link left_foot: geometry collision cylinder length=0.1 radius=0.02; visual cylinder length=0.1 radius=0.02
- link right_foot: geometry collision cylinder length=0.1 radius=0.02; visual cylinder length=0.1 radius=0.02
Joints:
- removed joint base_to_torso_joint
- joint left_forearm_pitch_joint: type revolute -> fixed
- joint left_shoulder_pitch_joint: type revolute -> fixed
- joint left_shoulder_yaw_joint: type revolute -> fixed
- joint right_forearm_pitch_joint: type revolute -> fixed
- joint right_shoulder_pitch_joint: type revolute -> fixed
- joint right_shoulder_yaw_joint: type revolute -> fixed

File: resources/robots/hopper/urdf/hopper.urdf (robot description, URDF)
Before this commit: robot 3D_hopper, 5 links, 4 joints
Links:
- link torso: geometry collision cylinder length=0.10000 radius=0.05000; visual cylinder length=0.10000 radius=0.05000
- link wheel1: geometry collision cylinder length=0.02000 radius=0.05000; visual cylinder length=0.02000 radius=0.05000
- link wheel2: geometry collision cylinder length=0.02000 radius=0.05000; visual cylinder length=0.02000 radius=0.05000
- link wheel3: geometry collision cylinder length=0.02000 radius=0.05000; visual cylinder length=0.02000 radius=0.05000
