Commit message: Hopper actuator frame fixed.

File: resources/robots/hopper/urdf/hopper.urdf (robot description, URDF)
Before this commit: robot 3D_hopper, 5 links, 4 joints
Joints:
- joint wheel1_rotation: origin xyz=0.0776 0 0.0547 rpy=0 0.5 0 -> xyz=0.0776 0 0.0547 rpy=0 0.9553 0
- joint wheel2_rotation: origin xyz=-0.0388 0.0672 0.0548 rpy=-0.5 -0.5 0 -> xyz=-0.0388 0.0672 0.0548 rpy=-0.87 -0.4 0
- joint wheel3_rotation: origin xyz=-0.0388 -0.0672 0.0548 rpy=0.5 -0.5 0 -> xyz=-0.0388 -0.0672 0.0548 rpy=0.87 -0.4 0

Commit message: Hopper attempts

File: resources/robots/hopper/urdf/hopper.urdf (robot description, URDF)
Before this commit: robot 3D_hopper, 5 links, 4 joints
Joints:
- joint wheel1_rotation: limit effort=1.6 velocity=600 -> effort=2.1 velocity=600
- joint wheel2_rotation: limit effort=1.6 velocity=600 -> effort=2.1 velocity=600
- joint wheel3_rotation: limit effort=1.6 velocity=600 -> effort=2.1 velocity=600

Commit message: Hopper Sim2Sim evaluation

File: resources/robots/hopper/urdf/hopper.urdf (robot description, URDF)
Before this commit: robot 3D_hopper, 5 links, 4 joints
Joints:
- joint foot_slide: limit lower=0 upper=0.1 effort=300 velocity=10 -> lower=0 upper=0.1 effort=25000 velocity=100; origin xyz=0.00000 0.00000 -0.2 -> xyz=0.00000 0.00000 -0.36

Commit message: After submission.

File: resources/robots/hopper/urdf/hopper.urdf (robot description, URDF)
Before this commit: robot 3D_hopper, 5 links, 4 joints
Links:
- link foot: geometry collision sphere radius=0.02000; visual mesh filename=../meshes/foot.stl scale=0.001 0.001 0.001
- link torso: geometry collision cylinder length=0.10000 radius=0.05000; visual mesh filename=../meshes/torso_reduced.stl scale=0.001 0.001 0.001
- link wheel1: geometry collision cylinder length=0.02000 radius=0.05000; visual mesh filename=../meshes/wheel_reduced.stl scale=0.001 0.001 0.001
- link wheel2: geometry collision cylinder length=0.02000 radius=0.05000; visual mesh filename=../meshes/wheel_reduced.stl scale=0.001 0.001 0.001
- link wheel3: geometry collision cylinder length=0.02000 radius=0.05000; visual mesh filename=../meshes/wheel_reduced.stl scale=0.001 0.001 0.001
Joints:
- joint wheel1_rotation: limit effort=2.1 velocity=600 -> lower=-7 upper=7 effort=2.1 velocity=600
- joint wheel2_rotation: limit effort=2.1 velocity=600 -> lower=-7 upper=7 effort=2.1 velocity=600
- joint wheel3_rotation: limit effort=2.1 velocity=600 -> lower=-7 upper=7 effort=2.1 velocity=600
